Commit message: :construction: <updated> added physics all the manipulator links and motors

File: cluerosity_description/urdf/cluerosity_links.xacro (robot description, xacro)
@@ -206,3 +206,25 @@
         </joint>
     </xacro:macro>
+    <xacro:macro name="motor_link" params="name joint_xyz joint_rpy parent axis_xyz axis_rpy lower upper">
+        <link name="${name}">
+            <xacro:mesh_link
+                xyz="0 0 0" rpy="0 0 0"
+                mesh_name="${motor}"/>
+            <xacro:box_collision
+                xyz="0 0 0" rpy="0 0 0"
+                box_size="0.065 0.065 0.1"/>
+            <xacro:link_inertia
+                xyz="0 0 0" rpy="0 0 0"
+                mass="0.33104028"
+                ixx="0.00022976" ixy="0" ixz="0"
+                iyy="0.00022976" iyz="0" izz="0.00011672"/>
+        </link>
+        <joint name="${name}_joint" type="revolute">
+            <parent link="${parent}" />
+            <child link="${name}" />
+            <origin xyz="${joint_xyz}" rpy="${joint_rpy}" />
+            <axis xyz="${axis_xyz}" rpy="${axis_rpy}" />
+            <limit effort="1000.0" lower="${lower}" upper="${upper}" velocity="0.5" /> -->
+        </joint>
+    </xacro:macro>
 </robot>

File: cluerosity_description/urdf/cluerosity_manipulator.xacro (robot description, xacro)
@@ -8,16 +8,10 @@
         +=======================+
     -->
-    <xacro:revolute_link
+    <xacro:motor_link
     name="motor_01"
-    link_xyz="0 0 0" link_rpy="0 0 0"
-    mesh_name="${motor}"
     joint_xyz="0.498 0.15 0.09" joint_rpy="${PI} 0 0"
     parent="base_link"
-    collision_xyz="0 0 0" collision_rpy="0 0 0" collision_size="0.105 0.105 0.075"
-    mass="0.61826506"
-    ixx="0.00067265" ixy="0" ixz="0"
-    iyy="0.0006728" iyz="0" izz="0.00080351"
     axis_xyz="0 0 1" axis_rpy="0 0 0"
-    lower="-0.35" upper="1.20"/>
+    lower="-0.3" upper="1.20"/>
     <xacro:fixed_link
     name="motor_connector_01"
@@ -26,18 +20,12 @@
     joint_xyz="0.046 0 0.0395" joint_rpy="${PI/2} ${PI/2} 0"
     parent="motor_01"
-    collision_xyz="0 0 0" collision_rpy="0 0 0" collision_size="0.105 0.105 0.075"
-    mass="0.61826506"
-    ixx="0.00067265" ixy="0" ixz="0"
-    iyy="0.0006728" iyz="0" izz="0.00080351"/>
-    <xacro:revolute_link
+    collision_xyz="0 0 0" collision_rpy="0 0 0" collision_size="0.05 0.05 0.05"
+    mass="0.1226583"
+    ixx="0.00006619" ixy="0" ixz="0"
+    iyy="0.00007979" iyz="0" izz="0.00006619"/>
+    <xacro:motor_link
     name="motor_02"
-    link_xyz="0 0 0" link_rpy="0 0 0"
-    mesh_name="${motor}"
     joint_xyz="0 0.036 -0.0395" joint_rpy="0 0 0"
     parent="motor_connector_01"
-    collision_xyz="0 0 0" collision_rpy="0 0 0" collision_size="0.105 0.105 0.075"
-    mass="0.61826506"
-    ixx="0.00067265" ixy="0" ixz="0"
-    iyy="0.0006728" iyz="0" izz="0.00080351"
     axis_xyz="0 0 1" axis_rpy="0 0 0"
     lower="${-PI/2}" upper="0"/>
@@ -48,18 +36,12 @@
     joint_xyz="0 0 0" joint_rpy="0 0 ${PI}"
     parent="motor_02"
-    collision_xyz="0 0 0" collision_rpy="0 0 0" collision_size="0.105 0.105 0.075"
-    mass="0.61826506"
-    ixx="0.00067265" ixy="0" ixz="0"
-    iyy="0.0006728" iyz="0" izz="0.00080351"/>
-    <xacro:revolute_link
+    collision_xyz="0 -0.180 0" collision_rpy="0 0 0" collision_size="0.06 0.36 0.06"
+    mass="1.28482853"
+    ixx="0.01710143" ixy="0" ixz="0"
+    iyy="0.00045593" iyz="0" izz="0.01705674"/>
+    <xacro:motor_link
     name="motor_03"
-    link_xyz="0 0 0" link_rpy="0 0 0"
-    mesh_name="${motor}"
     joint_xyz="0 -0.35 0" joint_rpy="0 0 0"
     parent="link_01"
-    collision_xyz="0 0 0" collision_rpy="0 0 0" collision_size="0.105 0.105 0.075"
-    mass="0.61826506"
-    ixx="0.00067265" ixy="0" ixz="0"
-    iyy="0.0006728" iyz="0" izz="0.00080351"
     axis_xyz="0 0 1" axis_rpy="0 0 0"
     lower="0" upper="${PI/2}"/>
@@ -70,18 +52,12 @@
     joint_xyz="0 0 0.0395" joint_rpy="0 0 ${PI}"
     parent="motor_03"
-    collision_xyz="0 0 0" collision_rpy="0 0 0" collision_size="0.105 0.105 0.075"
-    mass="0.61826506"
-    ixx="0.00067265" ixy="0" ixz="0"
-    iyy="0.0006728" iyz="0" izz="0.00080351"/>
-    <xacro:revolute_link
+    collision_xyz="0.180 0 0" collision_rpy="0 0 0" collision_size="0.36 0.06 0.06"
+    mass="1.19702377"
+    ixx="0.00043777" ixy="0.00000865" ixz="0"
+    iyy="0.01364495" iyz="0" izz="0.01375154"/>
+    <xacro:motor_link
     name="motor_04"
-    link_xyz="0 0 0" link_rpy="0 0 0"
-    mesh_name="${motor}"
     joint_xyz="0.370 0 -0.0395" joint_rpy="0 0 0"
     parent="link_02"
-    collision_xyz="0 0 0" collision_rpy="0 0 0" collision_size="0.105 0.105 0.075"
-    mass="0.61826506"
-    ixx="0.00067265" ixy="0" ixz="0"
-    iyy="0.0006728" iyz="0" izz="0.00080351"
     axis_xyz="0 0 1" axis_rpy="0 0 0"
     lower="${-PI/2}" upper="${PI/2}"/>
@@ -92,8 +68,8 @@
     joint_xyz="0 0 0" joint_rpy="0 0 0"
     parent="motor_04"
-    collision_xyz="0 0 0" collision_rpy="0 0 0" collision_size="0.105 0.105 0.075"
-    mass="0.61826506"
-    ixx="0.00067265" ixy="0" ixz="0"
-    iyy="0.0006728" iyz="0" izz="0.00080351"/>
+    collision_xyz="0 0 0" collision_rpy="0 0 0" collision_size="0.05 0.05 0.05"
+    mass="0.32771971"
+    ixx="0.00031006" ixy="0" ixz="0"
+    iyy="0.00083377" iyz="0" izz="0.00055215"/>
     <xacro:continuous_link
     name="motor_05"
@@ -102,5 +78,5 @@
     joint_xyz="0.1395 0 0.1" joint_rpy="0 ${-PI/2} 0"
     parent="motor_connector_02"
-    collision_xyz="0 0 0" collision_rpy="0 0 0" collision_size="0.105 0.105 0.075"
+    collision_xyz="0 0 0" collision_rpy="0 0 0" collision_size="0.05 0.05 0.15"
     mass="0.61826506"
     ixx="0.00067265" ixy="0" ixz="0"
@@ -114,6 +90,6 @@
     parent="motor_05"
     collision_xyz="0 0 0" collision_rpy="0 0 0" collision_size="0.105 0.105 0.075"
-    mass="0.61826506"
-    ixx="0.00067265" ixy="0" ixz="0"
-    iyy="0.0006728" iyz="0" izz="0.00080351"/>
+    mass="0.30502898"
+    ixx="0.00027224" ixy="0" ixz="0"
+    iyy="0.00042032" iyz="0" izz="0.00020714"/>
 </robot>
