Commit message: :white_check_mark: <tested ok> completed the robot structure with camera gimble and lidar sensor

File: cluerosity_description/urdf/cluerosity.xacro (robot description, xacro)
@@ -90,3 +90,137 @@
         <axis xyz="0 1 0" rpy="0 0 0" />
     </joint>
+    <!-- The Camera, Laser Gimbal system  -->
+    <!-- Gimbal Base  -->
+    <link name="gimbal_base">
+        <visual>
+            <origin xyz="0 0 0" rpy="0 0 0" />
+            <geometry>
+                <box size="0.15 0.15 0.15" />
+            </geometry>
+            <material name="black">
+                <color rgba="0 0 0 1" />
+            </material>
+        </visual>
+    </link>
+    <joint name="gimbal_base_joint" type="fixed">
+        <parent link="base_link" />
+        <child link="gimbal_base" />
+        <origin xyz="0.20 -0.10 0.275" rpy="0 0 0" />
+    </joint>
+    <!-- Gimbal Pole  -->
+    <link name="gimbal_pole">
+        <visual>
+            <origin xyz="0 0 0" rpy="0 0 0" />
+            <geometry>
+                <cylinder radius="0.0375" length="0.4" />
+            </geometry>
+            <material name="white">
+                <color rgba="1 1 1 1" />
+            </material>
+        </visual>
+    </link>
+    <joint name="gimbal_pole_joint" type="fixed">
+        <parent link="gimbal_base" />
+        <child link="gimbal_pole" />
+        <origin xyz="0 0 0.125" rpy="0 0 0" />
+    </joint>
+    <!-- Gimbal Yaw Link -->
+    <link name="gimbal_yaw_link">
+        <visual>
+            <origin xyz="0 0 0" rpy="0 0 0" />
+            <geometry>
+                <cylinder radius="0.1" length="0.05" />
+            </geometry>
+            <material name="black">
+                <color rgba="0 0 0 1" />
+            </material>
+        </visual>
+    </link>
+    <joint name="gimbal_yaw_joint" type="continuous">
+        <parent link="gimbal_pole" />
+        <child link="gimbal_yaw_link" />
+        <origin xyz="0 0 0.15" rpy="0 0 0" />
+        <axis xyz="0 0 1" rpy="0 0 0" />
+    </joint>
+    <!-- Gimbal Sensor Housing  -->
+    <link name="gimbal_sensor_housing">
+        <visual>
+            <origin xyz="0 0 0" rpy="0 0 0" />
+            <geometry>
+                <box size="0.15 0.30 0.15" />
+            </geometry>
+            <material name="white">
+                <color rgba="1 1 1 1" />
+            </material>
+        </visual>
+        <visual>
+            <origin xyz="0.08 -0.05 0" rpy="0 1.5708 0" />
+            <geometry>
+                <cylinder radius="0.05" length="0.01" />
+            </geometry>
+            <material name="black">
+                <color rgba="0 0 0 1" />
+            </material>
+        </visual>
+    </link>
+    <joint name="gimbal_sensor_housing_joint" type="revolute">
+        <parent link="gimbal_yaw_link" />
+        <child link="gimbal_sensor_housing" />
+        <origin xyz="0 0 0.125" rpy="0 0 0" />
+        <axis xyz="0 1 0" rpy="0 0 0" />
+        <limit effort="1000.0" lower="-0.35" upper="0.35" velocity="0.5" />
+    </joint>
+    <!-- Velodyne LiDAR Sensor -->
+    <!-- Sensor Base -->
+    <link name="lidar_base">
+        <visual>
+            <origin xyz="0 0 0" rpy="0 0 0" />
+            <geometry>
+                <box size="0.12 0.12 0.12" />
+            </geometry>
+            <material name="black">
+                <color rgba="0 0 0 1" />
+            </material>
+        </visual>
+    </link>
+    <joint name="lidar_base_joint" type="fixed">
+        <parent link="base_link" />
+        <child link="lidar_base" />
+        <origin xyz="-0.215 0.115 0.26" rpy="0 0 0" />
+    </joint>
+    <!-- LiDAR Sensor -->
+    <link name="lidar_sensor">
+        <visual>
+            <origin xyz="0 0 0" rpy="0 0 0" />
+            <geometry>
+                <cylinder radius="0.0515" length="0.036" />
+            </geometry>
+            <material name="bluish">
+                <color rgba="0.1373 0.1961 0.6471 0.8" />
+            </material>
+        </visual>
+        <visual>
+            <origin xyz="0 0 0.027" rpy="0 0 0" />
+            <geometry>
+                <cylinder radius="0.0515" length="0.018" />
+            </geometry>
+            <material name="white">
+                <color rgba="1 1 1 1" />
+            </material>
+        </visual>
+        <visual>
+            <origin xyz="0 0 -0.027" rpy="0 0 0" />
+            <geometry>
+                <cylinder radius="0.0515" length="0.018" />
+            </geometry>
+            <material name="white">
+                <color rgba="1 1 1 1" />
+            </material>
+        </visual>
+    </link>
+    <joint name="lidar_sensor_joint" type="fixed">
+        <parent link="lidar_base" />
+        <child link="lidar_sensor" />
+        <origin xyz="0 0 0.096" rpy="0 0 0" />
+    </joint>
 </robot>

Commit message: :construction: <updated> added wheel, rim and robot base meshes to the robot urdf

File: cluerosity_description/urdf/cluerosity.xacro (robot description, xacro)
@@ -3,11 +3,15 @@
     <link name="base_link">
         <visual>
-            <origin rpy="0 0 0" xyz="0 0 0.1" />
-            <geometry>
-                <box size="0.6 0.4 0.2" />
-            </geometry>
-            <material name="cyan">
+            <origin rpy="0 3.14159265359 -1.5708" xyz="0 0 0.15" />
+            <geometry>
+                <!-- <box size="0.6 0.4 0.2" /> -->
+                <mesh filename="package://cluerosity_description/meshes/robot_base.dae" />
+            </geometry>
+            <!-- <material name="cyan">
                 <color rgba="0 1.0 1.0 1.0" />
-            </material>
+            </material> -->
+            <!-- <material name="white">
+                <color rgba="1 1 1 1" />
+            </material> -->
         </visual>
     </link>
@@ -19,15 +23,50 @@
         <child link="base_footprint" />
     </joint>
+    <link name="front_shaft">
+        <visual>
+            <origin rpy="1.5708 0 0" xyz="0 0 0" />
+            <geometry>
+                <cylinder radius="0.010" length="0.550" />
+            </geometry>
+            <material name="white">
+                <color rgba="1 1 1 1" />
+            </material>
+        </visual>
+    </link>
+    <joint name="front_shaft_joint" type="fixed">
+        <origin xyz="0.350 0 0.05" rpy="0 0 0" />
+        <parent link="base_link" />
+        <child link="front_shaft" />
+    </joint>
+    <link name="rear_shaft">
+        <visual>
+            <origin rpy="1.5708 0 0" xyz="0 0 0" />
+            <geometry>
+                <cylinder radius="0.010" length="0.550" />
+            </geometry>
+            <material name="white">
+                <color rgba="1 1 1 1" />
+            </material>
+        </visual>
+    </link>
+    <joint name="rear_shaft_joint" type="fixed">
+        <origin xyz="-0.20 0 0.05" rpy="0 0 0" />
+        <parent link="base_link" />
+        <child link="rear_shaft" />
+    </joint>
     <!-- Wheel definition -->
     <!-- RIGHT WHEEL  -->
     <link name="right_front_wheel">
-        <visual>
-            <origin xyz="0 0 0" rpy="1.5708 0 0" />
-            <geometry>
-                <cylinder radius="0.175" length="0.15" />
-            </geometry>
-            <material name="black">
-                <color rgba="0 0 0 1" />
-            </material>
+        <visual name="tyre">
+            <origin xyz="-0.14686986  0 0" rpy="1.5708 0 -1.5708" />
+            <geometry>
+                <mesh filename="package://cluerosity_description/meshes/tyre.dae" />
+            </geometry>
+        </visual>
+        <visual name="rim">
+            <origin xyz="0  0 0" rpy="0 0 0" />
+            <geometry>
+                <mesh filename="package://cluerosity_description/meshes/rim.dae" />
+            </geometry>
         </visual>
     </link>
@@ -35,16 +74,19 @@
         <parent link="base_link" />
         <child link="right_front_wheel" />
-        <origin xyz="0.3 -0.30 0.045" rpy="0 0 0" />
+        <origin xyz="0.35 -0.30 0.05" rpy="0 0 0" />
         <axis xyz="0 1 0" rpy="0 0 0" />
     </joint>
     <link name="right_back_wheel">
-        <visual>
-            <origin xyz="0 0 0" rpy="1.5708 0 0" />
-            <geometry>
-                <cylinder radius="0.175" length="0.15" />
-            </geometry>
-            <material name="black">
-                <color rgba="0 0 0 1" />
-            </material>
+        <visual name="tyre">
+            <origin xyz="-0.14686986  0 0" rpy="1.5708 0 -1.5708" />
+            <geometry>
+                <mesh filename="package://cluerosity_description/meshes/tyre.dae" />
+            </geometry>
+        </visual>
+        <visual name="rim">
+            <origin xyz="0  0 0" rpy="0 0 0" />
+            <geometry>
+                <mesh filename="package://cluerosity_description/meshes/rim.dae" />
+            </geometry>
         </visual>
     </link>
@@ -52,17 +94,20 @@
         <parent link="base_link" />
         <child link="right_back_wheel" />
-        <origin xyz="-0.3 -0.30 0.045" rpy="0 0 0" />
+        <origin xyz="-0.20 -0.30 0.05" rpy="0 0 0" />
         <axis xyz="0 1 0" rpy="0 0 0" />
     </joint>
     <!-- LEFT WHEEL -->
     <link name="left_front_wheel">
-        <visual>
-            <origin xyz="0 0 0" rpy="1.5708 0 0" />
-            <geometry>
-                <cylinder radius="0.175" length="0.15" />
-            </geometry>
-            <material name="black">
-                <color rgba="0 0 0 1" />
-            </material>
+        <visual name="tyre">
+            <origin xyz="-0.14686986  0 0" rpy="1.5708 0 -1.5708" />
+            <geometry>
+                <mesh filename="package://cluerosity_description/meshes/tyre.dae" />
+            </geometry>
+        </visual>
+        <visual name="rim">
+            <origin xyz="0  0 0" rpy="0 0 3.14159265359" />
+            <geometry>
+                <mesh filename="package://cluerosity_description/meshes/rim.dae" />
+            </geometry>
         </visual>
     </link>
@@ -70,16 +115,19 @@
         <parent link="base_link" />
         <child link="left_front_wheel" />
-        <origin xyz="0.3 0.30 0.045" rpy="0 0 0" />
+        <origin xyz="0.35 0.30 0.05" rpy="0 0 0" />
         <axis xyz="0 1 0" rpy="0 0 0" />
     </joint>
     <link name="left_back_wheel">
-        <visual>
-            <origin xyz="0 0 0" rpy="1.5708 0 0" />
-            <geometry>
-                <cylinder radius="0.175" length="0.15" />
-            </geometry>
-            <material name="black">
-                <color rgba="0 0 0 1" />
-            </material>
+        <visual name="tyre">
+            <origin xyz="-0.14686986  0 0" rpy="1.5708 0 -1.5708" />
+            <geometry>
+                <mesh filename="package://cluerosity_description/meshes/tyre.dae" />
+            </geometry>
+        </visual>
+        <visual name="rim">
+            <origin xyz="0  0 0" rpy="0 0 3.14159265359" />
+            <geometry>
+                <mesh filename="package://cluerosity_description/meshes/rim.dae" />
+            </geometry>
         </visual>
     </link>
@@ -87,10 +135,10 @@
         <parent link="base_link" />
         <child link="left_back_wheel" />
-        <origin xyz="-0.3 0.30 0.045" rpy="0 0 0" />
+        <origin xyz="-0.20 0.30 0.05" rpy="0 0 0" />
         <axis xyz="0 1 0" rpy="0 0 0" />
     </joint>
     <!-- The Camera, Laser Gimbal system  -->
     <!-- Gimbal Base  -->
-    <link name="gimbal_base">
+    <!-- <link name="gimbal_base">
         <visual>
             <origin xyz="0 0 0" rpy="0 0 0" />
@@ -107,7 +155,7 @@
         <child link="gimbal_base" />
         <origin xyz="0.20 -0.10 0.275" rpy="0 0 0" />
-    </joint>
+    </joint> -->
     <!-- Gimbal Pole  -->
-    <link name="gimbal_pole">
+    <!-- <link name="gimbal_pole">
         <visual>
             <origin xyz="0 0 0" rpy="0 0 0" />
@@ -124,7 +172,7 @@
         <child link="gimbal_pole" />
         <origin xyz="0 0 0.125" rpy="0 0 0" />
-    </joint>
+    </joint> -->
     <!-- Gimbal Yaw Link -->
-    <link name="gimbal_yaw_link">
+    <!-- <link name="gimbal_yaw_link">
         <visual>
             <origin xyz="0 0 0" rpy="0 0 0" />
@@ -142,7 +190,7 @@
         <origin xyz="0 0 0.15" rpy="0 0 0" />
         <axis xyz="0 0 1" rpy="0 0 0" />
-    </joint>
+    </joint> -->
     <!-- Gimbal Sensor Housing  -->
-    <link name="gimbal_sensor_housing">
+    <!-- <link name="gimbal_sensor_housing">
         <visual>
             <origin xyz="0 0 0" rpy="0 0 0" />
@@ -170,8 +218,8 @@
         <axis xyz="0 1 0" rpy="0 0 0" />
         <limit effort="1000.0" lower="-0.35" upper="0.35" velocity="0.5" />
-    </joint>
+    </joint> -->
     <!-- Velodyne LiDAR Sensor -->
     <!-- Sensor Base -->
-    <link name="lidar_base">
+    <!-- <link name="lidar_base">
         <visual>
             <origin xyz="0 0 0" rpy="0 0 0" />
@@ -188,7 +236,7 @@
         <child link="lidar_base" />
         <origin xyz="-0.215 0.115 0.26" rpy="0 0 0" />
-    </joint>
+    </joint> -->
     <!-- LiDAR Sensor -->
-    <link name="lidar_sensor">
+    <!-- <link name="lidar_sensor">
         <visual>
             <origin xyz="0 0 0" rpy="0 0 0" />
@@ -223,4 +271,4 @@
         <child link="lidar_sensor" />
         <origin xyz="0 0 0.096" rpy="0 0 0" />
-    </joint>
+    </joint> -->
 </robot>

Commit message: :construction: <updated> added the velodyne lidar mesh to the urdf

File: cluerosity_description/urdf/cluerosity.xacro (robot description, xacro)
@@ -221,13 +221,10 @@
     <!-- Velodyne LiDAR Sensor -->
     <!-- Sensor Base -->
-    <!-- <link name="lidar_base">
-        <visual>
-            <origin xyz="0 0 0" rpy="0 0 0" />
-            <geometry>
-                <box size="0.12 0.12 0.12" />
-            </geometry>
-            <material name="black">
-                <color rgba="0 0 0 1" />
-            </material>
+    <link name="lidar_base">
+        <visual>
+            <origin xyz="-0.075 0 0.05" rpy="0 3.14159265359 1.5708" />
+            <geometry>
+                <mesh filename="package://cluerosity_description/meshes/lidar_base.dae" />
+            </geometry>
         </visual>
     </link>
@@ -235,34 +232,13 @@
         <parent link="base_link" />
         <child link="lidar_base" />
-        <origin xyz="-0.215 0.115 0.26" rpy="0 0 0" />
-    </joint> -->
+        <origin xyz="-0.325 0.140 0.25" rpy="0 0 0" />
+    </joint>
     <!-- LiDAR Sensor -->
-    <!-- <link name="lidar_sensor">
-        <visual>
-            <origin xyz="0 0 0" rpy="0 0 0" />
-            <geometry>
-                <cylinder radius="0.0515" length="0.036" />
-            </geometry>
-            <material name="bluish">
-                <color rgba="0.1373 0.1961 0.6471 0.8" />
-            </material>
-        </visual>
-        <visual>
-            <origin xyz="0 0 0.027" rpy="0 0 0" />
-            <geometry>
-                <cylinder radius="0.0515" length="0.018" />
-            </geometry>
-            <material name="white">
-                <color rgba="1 1 1 1" />
-            </material>
-        </visual>
-        <visual>
-            <origin xyz="0 0 -0.027" rpy="0 0 0" />
-            <geometry>
-                <cylinder radius="0.0515" length="0.018" />
-            </geometry>
-            <material name="white">
-                <color rgba="1 1 1 1" />
-            </material>
+    <link name="lidar_sensor">
+        <visual>
+            <origin xyz="0 0 0" rpy="0 0 0" />
+            <geometry>
+                <mesh filename="package://cluerosity_description/meshes/velodyne_lidar.dae" />
+            </geometry>
         </visual>
     </link>
@@ -270,5 +246,5 @@
         <parent link="lidar_base" />
         <child link="lidar_sensor" />
-        <origin xyz="0 0 0.096" rpy="0 0 0" />
-    </joint> -->
+        <origin xyz="-0.2 0 0.05" rpy="0 0 0" />
+    </joint>
 </robot>

Commit message: :white_check_mark: <tested ok> completed version 0.1 of cluerosity robot

File: cluerosity_description/urdf/cluerosity.xacro (robot description, xacro)
@@ -5,13 +5,6 @@
             <origin rpy="0 3.14159265359 -1.5708" xyz="0 0 0.15" />
             <geometry>
-                <!-- <box size="0.6 0.4 0.2" /> -->
                 <mesh filename="package://cluerosity_description/meshes/robot_base.dae" />
             </geometry>
-            <!-- <material name="cyan">
-                <color rgba="0 1.0 1.0 1.0" />
-            </material> -->
-            <!-- <material name="white">
-                <color rgba="1 1 1 1" />
-            </material> -->
         </visual>
     </link>
@@ -140,83 +133,65 @@
     <!-- The Camera, Laser Gimbal system  -->
     <!-- Gimbal Base  -->
-    <!-- <link name="gimbal_base">
+    <link name="gimbal_base">
+        <visual>
+            <origin xyz="0 0 0.025" rpy="0 0 0" />
+            <geometry>
+                <box size="0.1 0.1 0.05" />
+            </geometry>
+            <material name="dark_gray">
+                <color rgba="0.35 0.38 0.4 1" />
+            </material>
+        </visual>
+    </link>
+    <joint name="gimbal_base_joint" type="fixed">
+        <parent link="base_link" />
+        <child link="gimbal_base" />
+        <origin xyz="0.340 -0.140 0.1" rpy="0 0 1.5708" />
+    </joint>
+    <!-- Gimbal Axle  -->
+    <link name="gimbal_axle">
         <visual>
             <origin xyz="0 0 0" rpy="0 0 0" />
             <geometry>
-                <box size="0.15 0.15 0.15" />
-            </geometry>
-            <material name="black">
-                <color rgba="0 0 0 1" />
-            </material>
-        </visual>
-    </link>
-    <joint name="gimbal_base_joint" type="fixed">
-        <parent link="base_link" />
-        <child link="gimbal_base" />
-        <origin xyz="0.20 -0.10 0.275" rpy="0 0 0" />
-    </joint> -->
-    <!-- Gimbal Pole  -->
-    <!-- <link name="gimbal_pole">
-        <visual>
-            <origin xyz="0 0 0" rpy="0 0 0" />
-            <geometry>
-                <cylinder radius="0.0375" length="0.4" />
-            </geometry>
-            <material name="white">
-                <color rgba="1 1 1 1" />
-            </material>
-        </visual>
-    </link>
-    <joint name="gimbal_pole_joint" type="fixed">
+                <mesh filename="package://cluerosity_description/meshes/gimbal_axle.dae" />
+            </geometry>
+        </visual>
+    </link>
+    <joint name="gimbal_axle_joint" type="continuous">
         <parent link="gimbal_base" />
-        <child link="gimbal_pole" />
-        <origin xyz="0 0 0.125" rpy="0 0 0" />
-    </joint> -->
-    <!-- Gimbal Yaw Link -->
-    <!-- <link name="gimbal_yaw_link">
-        <visual>
-            <origin xyz="0 0 0" rpy="0 0 0" />
-            <geometry>
-                <cylinder radius="0.1" length="0.05" />
-            </geometry>
-            <material name="black">
-                <color rgba="0 0 0 1" />
-            </material>
-        </visual>
-    </link>
-    <joint name="gimbal_yaw_joint" type="continuous">
-        <parent link="gimbal_pole" />
-        <child link="gimbal_yaw_link" />
-        <origin xyz="0 0 0.15" rpy="0 0 0" />
+        <child link="gimbal_axle" />
+        <origin xyz="0 0 0" rpy="0 0 0" />
         <axis xyz="0 0 1" rpy="0 0 0" />
-    </joint> -->
+    </joint>
+    <!-- Stepper Motor  -->
+    <link name="stepper_motor">
+        <visual>
+            <origin xyz="0 0 0" rpy="0 1.5708 0" />
+            <geometry>
+                <mesh filename="package://cluerosity_description/meshes/stepper_motor.dae" />
+            </geometry>
+        </visual>
+    </link>
+    <joint name="stepper_motor_joint" type="fixed">
+        <parent link="gimbal_axle" />
+        <child link="stepper_motor" />
+        <origin xyz="-0.10 0 0.19" rpy="0 0 0" />
+    </joint>
     <!-- Gimbal Sensor Housing  -->
-    <!-- <link name="gimbal_sensor_housing">
-        <visual>
-            <origin xyz="0 0 0" rpy="0 0 0" />
-            <geometry>
-                <box size="0.15 0.30 0.15" />
-            </geometry>
-            <material name="white">
-                <color rgba="1 1 1 1" />
-            </material>
-        </visual>
-        <visual>
-            <origin xyz="0.08 -0.05 0" rpy="0 1.5708 0" />
-            <geometry>
-                <cylinder radius="0.05" length="0.01" />
-            </geometry>
-            <material name="black">
-                <color rgba="0 0 0 1" />
-            </material>
-        </visual>
-    </link>
-    <joint name="gimbal_sensor_housing_joint" type="revolute">
-        <parent link="gimbal_yaw_link" />
-        <child link="gimbal_sensor_housing" />
-        <origin xyz="0 0 0.125" rpy="0 0 0" />
-        <axis xyz="0 1 0" rpy="0 0 0" />
+    <link name="sensor_housing">
+        <visual>
+            <origin xyz="0 0 0.053" rpy="0 0 0" />
+            <geometry>
+                <mesh filename="package://cluerosity_description/meshes/sensor_housing.dae" />
+            </geometry>
+        </visual>
+    </link>
+    <joint name="sensor_housing_joint" type="revolute">
+        <parent link="stepper_motor" />
+        <child link="sensor_housing" />
+        <origin xyz="0.122 0 0" rpy="0 0 0" />
+        <axis xyz="1 0 0" rpy="0 0 0" />
         <limit effort="1000.0" lower="-0.35" upper="0.35" velocity="0.5" />
-    </joint> -->
+    </joint>
     <!-- Velodyne LiDAR Sensor -->
     <!-- Sensor Base -->
