Commit message: :recycle: <refactored> rewrote and reorganized the xacro macros for modularity and clarity

File: cluerosity_description/urdf/cluerosity.xacro (robot description, xacro)
@@ -3,9 +3,11 @@
     <!-- Includes -->
     <xacro:include filename="$(find cluerosity_description)/urdf/meshes.xacro" />
+    <xacro:include filename="$(find cluerosity_description)/urdf/materials.xacro" />
+    <xacro:include filename="$(find cluerosity_description)/urdf/visual.xacro" />
+    <xacro:include filename="$(find cluerosity_description)/urdf/physics.xacro" />
     <xacro:include filename="$(find cluerosity_description)/urdf/wheels.xacro" />
-    <xacro:include filename="$(find cluerosity_description)/urdf/sensor_gimbal.xacro" />
     <xacro:include filename="$(find cluerosity_description)/urdf/cluerosity_links.xacro" />
     <!-- Properties -->
-    <xacro:property name="pi" value="3.14159265359" />
+    <xacro:property name="PI" value="3.14159265359" />
     <!--
         +=====================+
@@ -13,5 +15,5 @@
         +=====================+
     -->
-    <xacro:base_link/>
+    <xacro:base_link mesh_name="${robot_base}"/>
     <!--
         +=====================+
@@ -33,5 +35,5 @@
     <xacro:cluerosity_wheel
         name="right_front_wheel"
-        tyre_xyz="-0.14686986 0 0" tyre_rpy="${pi/2} 0 ${-pi/2}"
+        tyre_xyz="-0.14686986 0 0" tyre_rpy="${PI/2} 0 ${-PI/2}"
         rim_xyz="0 0 0" rim_rpy="0 0 0"
         joint_xyz="0.35 -0.30 0.05" joint_rpy="0 0 0" />
@@ -39,5 +41,5 @@
     <xacro:cluerosity_wheel
         name="right_rear_wheel"
-        tyre_xyz="-0.14686986 0 0" tyre_rpy="${pi/2} 0 ${-pi/2}"
+        tyre_xyz="-0.14686986 0 0" tyre_rpy="${PI/2} 0 ${-PI/2}"
         rim_xyz="0 0 0" rim_rpy="0 0 0"
         joint_xyz="-0.20 -0.30 0.05" joint_rpy="0 0 0" />
@@ -45,12 +47,12 @@
     <xacro:cluerosity_wheel
         name="left_front_wheel"
-        tyre_xyz="-0.14686986 0 0" tyre_rpy="${pi/2} 0 ${-pi/2}"
-        rim_xyz="0 0 0" rim_rpy="0 0 ${pi}"
+        tyre_xyz="-0.14686986 0 0" tyre_rpy="${PI/2} 0 ${-PI/2}"
+        rim_xyz="0 0 0" rim_rpy="0 0 ${PI}"
         joint_xyz="0.35 0.30 0.05" joint_rpy="0 0 0" />
     <!-- Left Rear Wheel -->
     <xacro:cluerosity_wheel
         name="left_rear_wheel"
-        tyre_xyz="-0.14686986 0 0" tyre_rpy="${pi/2} 0 ${-pi/2}"
-        rim_xyz="0 0 0" rim_rpy="0 0 ${pi}"
+        tyre_xyz="-0.14686986 0 0" tyre_rpy="${PI/2} 0 ${-PI/2}"
+        rim_xyz="0 0 0" rim_rpy="0 0 ${PI}"
         joint_xyz="-0.20 0.30 0.05" joint_rpy="0 0 0" />
     <!--
@@ -62,11 +64,11 @@
     <xacro:gimbal_base />
     <!-- Gimbal Axle  -->
-    <xacro:gimbal_axle />
+    <xacro:gimbal_axle mesh_name="${gimbal_axle}"/>
     <!-- Gimbal Sensor Housing  -->
-    <xacro:sensor_housing />
+    <xacro:sensor_housing mesh_name="${sensor_housing}" />
     <!-- Stepper Motor -->
     <xacro:fixed_link
         name="stepper_motor"
-        link_xyz="0 0 0" link_rpy="0 ${pi/2} 0"
+        link_xyz="0 0 0" link_rpy="0 ${PI/2} 0"
         mesh_name="${stepper_motor}"
         joint_xyz="-0.10 0 0.19" joint_rpy="0 0 0"
@@ -80,5 +82,5 @@
     <xacro:fixed_link
         name="lidar_base"
-        link_xyz="-0.075 0 0.05" link_rpy="0 ${pi} ${pi/2}"
+        link_xyz="-0.075 0 0.05" link_rpy="0 ${PI} ${PI/2}"
         mesh_name="${lidar_base}"
         joint_xyz="-0.325 0.140 0.25" joint_rpy="0 0 0"

File: cluerosity_description/urdf/cluerosity_links.xacro (robot description, xacro)
@@ -1,5 +1,4 @@
+<?xml version="1.0"?>
 <robot xmlns:xacro="http://ros.org/wiki/xacro">
-    <xacro:include filename="$(find cluerosity_description)/urdf/materials.xacro" />
-    <xacro:include filename="$(find cluerosity_description)/urdf/physics.xacro" />
     <!--
         +===========================+
@@ -9,10 +8,7 @@
     <xacro:macro name="fixed_link" params="name link_xyz link_rpy mesh_name joint_xyz joint_rpy parent">
         <link name="${name}">
-            <visual>
-                <origin xyz="${link_xyz}" rpy="${link_rpy}" />
-                <geometry>
-                    <mesh filename="${mesh_name}" />
-                </geometry>
-            </visual>
+            <xacro:mesh_link
+                xyz="${link_xyz}" rpy="${link_rpy}"
+                mesh_name="${mesh_name}"/>
         </link>
         <joint name="${name}_joint" type="fixed">
@@ -23,37 +19,13 @@
     </xacro:macro>
     <!--
-        +=============================+
-        |      Wheel Shaft Macro      |
-        +============================+
-    -->
-    <xacro:macro name="cluerosity_shaft" params="name joint_xyz">
-        <link name="${name}">
-            <visual>
-                <origin xyz="0 0 0" rpy="${pi/2} 0 0" />
-                <geometry>
-                    <cylinder radius="0.010" length="0.550" />
-                </geometry>
-                <material name="white" />
-            </visual>
-        </link>
-        <joint name="${name}_joint" type="fixed">
-            <parent link="base_link" />
-            <child link="${name}" />
-            <origin xyz="${joint_xyz}" rpy="0 0 0" />
-        </joint>
-    </xacro:macro>
-    <!--
         +==============================================+
         |      Base Link and Base footprint Macro      |
         +==============================================+
     -->
-    <xacro:macro name="base_link">
+    <xacro:macro name="base_link" params="mesh_name">
         <link name="base_link">
-            <visual>
-                <origin rpy="0 ${pi} ${-pi/2}" xyz="0 0 0.15" />
-                <geometry>
-                    <mesh filename="${robot_base}" />
-                </geometry>
-            </visual>
+            <xacro:mesh_link
+                xyz="0 0 0.15" rpy="0 ${PI} ${-PI/2}"
+                mesh_name="${mesh_name}"/>
             <xacro:box_collision
                 xyz="0 0 0.075" rpy="0 0 0"
@@ -79,3 +51,51 @@
         </joint>
     </xacro:macro>
+    <!--
+        +==================================+
+        |   Sensor Gimbal links Macro     |
+        +================================+
+    -->
+    <!-- Gimbal Base  -->
+    <xacro:macro name="gimbal_base">
+        <link name="gimbal_base">
+            <xacro:box_link
+                xyz="0 0 0.025" rpy="0 0 0"
+                box_size="0.1 0.1 0.05"
+                material_name="dark_gray"/>
+        </link>
+        <joint name="gimbal_base_joint" type="fixed">
+            <parent link="base_link" />
+            <child link="gimbal_base" />
+            <origin xyz="0.340 -0.140 0.1" rpy="0 0 ${PI/2}" />
+        </joint>
+    </xacro:macro>
+    <!-- Gimbal Axle -->
+    <xacro:macro name="gimbal_axle" params="mesh_name">
+        <link name="gimbal_axle">
+            <xacro:mesh_link
+                xyz="0 0 0" rpy="0 0 0"
+                mesh_name="${mesh_name}"/>
+        </link>
+        <joint name="gimbal_axle_joint" type="continuous">
+            <parent link="gimbal_base" />
+            <child link="gimbal_axle" />
+            <origin xyz="0 0 0" rpy="0 0 0" />
+            <axis xyz="0 0 1" rpy="0 0 0" />
+        </joint>
+    </xacro:macro>
+    <!-- Sensor Housing -->
+    <xacro:macro name="sensor_housing" params="mesh_name">
+        <link name="sensor_housing">
+            <xacro:mesh_link
+                xyz="0 0 0.053" rpy="0 0 0"
+                mesh_name="${mesh_name}"/>
+        </link>
+        <joint name="sensor_housing_joint" type="revolute">
+            <parent link="stepper_motor" />
+            <child link="sensor_housing" />
+            <origin xyz="0.122 0 0" rpy="0 0 0" />
+            <axis xyz="1 0 0" rpy="0 0 0" />
+            <limit effort="1000.0" lower="-0.35" upper="0.35" velocity="0.5" />
+        </joint>
+    </xacro:macro>
 </robot>

File: cluerosity_description/urdf/materials.xacro (robot description, xacro)
@@ -25,4 +25,7 @@
         <color rgba="1.0 1.0 1.0 1.0" />
     </material>
+    <material name="dark_gray">
+        <color rgba="0.35 0.38 0.4 1" />
+    </material>
     <material name="cyan">
         <color rgba="0 1.0 1.0 1.0" />

File: cluerosity_description/urdf/physics.xacro (robot description, xacro)
@@ -1,3 +1,5 @@
+<?xml version="1.0"?>
 <robot xmlns:xacro="http://ros.org/wiki/xacro">
+    <!-- Box Collsion -->
     <xacro:macro name="box_collision" params="xyz rpy box_size">
         <collision>
@@ -8,4 +10,5 @@
         </collision>
     </xacro:macro>
+    <!-- Cylindrical Collision  -->
     <xacro:macro name="cylinder_collision" params="xyz rpy length radius">
         <collision>
@@ -16,4 +19,5 @@
         </collision>
     </xacro:macro>
+    <!-- Mass Properties: Inertial definition -->
     <xacro:macro name="link_inertia" params="xyz rpy mass ixx ixy ixz iyy iyz izz">
         <inertial>

File: cluerosity_description/urdf/visual.xacro (robot description, xacro)
@@ -1,4 +1,5 @@
+<?xml version="1.0"?>
 <robot xmlns:xacro="http://ros.org/wiki/xacro">
-    <xacro:include filename="$(find cluerosity_description)/urdf/materials.xacro" />
+    <!-- For Links with Meshes -->
     <xacro:macro name="mesh_link" params="xyz rpy mesh_name">
         <visual>
@@ -9,4 +10,5 @@
         </visual>
     </xacro:macro>
+    <!-- For Cylindrical Links  -->
     <xacro:macro name="cylinder_link" params="xyz rpy length radius material_name">
         <visual>
@@ -18,4 +20,5 @@
         </visual>
     </xacro:macro>
+    <!-- For box links -->
     <xacro:macro name="box_link" params="xyz rpy box_size material_name">
         <visual>

File: cluerosity_description/urdf/wheels.xacro (robot description, xacro)
@@ -1,21 +1,25 @@
+<?xml version="1.0"?>
 <robot xmlns:xacro="http://ros.org/wiki/xacro">
-    <!-- Includes -->
-    <xacro:include filename="$(find cluerosity_description)/urdf/meshes.xacro" />
-    <xacro:include filename="$(find cluerosity_description)/urdf/wheel_physics.xacro" />
+    <!--
+        +==================================+
+        |      Wheel Definition Macro      |
+        +=================================+
+    -->
     <xacro:macro name="cluerosity_wheel" params="name tyre_xyz tyre_rpy rim_xyz rim_rpy joint_xyz joint_rpy">
         <link name="${name}">
-            <visual name="tyre">
-                <origin xyz="${tyre_xyz}" rpy="${tyre_rpy}" />
-                <geometry>
-                    <mesh filename="${tyre}" />
-                </geometry>
-            </visual>
-            <visual name="rim">
-                <origin xyz="${rim_xyz}" rpy="${rim_rpy}" />
-                <geometry>
-                    <mesh filename="${rim}" />
-                </geometry>
-            </visual>
-            <xacro:wheel_physics />
+            <xacro:mesh_link
+                xyz="${tyre_xyz}" rpy="${tyre_rpy}"
+                mesh_name="${tyre}"/>
+            <xacro:mesh_link
+                xyz="${rim_xyz}" rpy="${rim_rpy}"
+                mesh_name="${rim}"/>
+            <xacro:cylinder_collision
+                xyz="0 0 0" rpy="${PI/2} 0 0"
+                length="0.15" radius="0.165" />
+            <xacro:link_inertia
+                xyz="0 0 0" rpy="${PI/2} 0 0"
+                mass="5.52250093"
+                ixx="0.13326254" ixy="0" ixz="0"
+                iyy="0.07660474" iyz="0"  izz="0.077"/>
         </link>
         <joint name="${name}_joint" type="continuous">
@@ -26,3 +30,21 @@
         </joint>
     </xacro:macro>
+    <!--
+        +=============================+
+        |      Wheel Shaft Macro      |
+        +============================+
+    -->
+    <xacro:macro name="cluerosity_shaft" params="name joint_xyz">
+        <link name="${name}">
+            <xacro:cylinder_link
+                xyz="0 0 0" rpy="${PI/2} 0 0"
+                radius="0.010" length="0.550"
+                material_name="white"/>
+        </link>
+        <joint name="${name}_joint" type="fixed">
+            <parent link="base_link" />
+            <child link="${name}" />
+            <origin xyz="${joint_xyz}" rpy="0 0 0" />
+        </joint>
+    </xacro:macro>
 </robot>

Commit message: :construction: <updated> added physics to every link of the robot

File: cluerosity_description/urdf/cluerosity.xacro (robot description, xacro)
@@ -73,5 +73,9 @@
         mesh_name="${stepper_motor}"
         joint_xyz="-0.10 0 0.19" joint_rpy="0 0 0"
-        parent="gimbal_axle" />
+        parent="gimbal_axle"
+        collision_xyz="0.0325 0 0" collision_rpy="0 ${PI/2} 0" collision_size="0.05 0.05 0.080"
+        mass="0.20879833"
+        ixx="0.0000978" ixy="0" ixz="0"
+        iyy="0.0000978" iyz="0" izz="0.0000491"/>
     <!--
         +=======================+
@@ -85,5 +89,9 @@
         mesh_name="${lidar_base}"
         joint_xyz="-0.325 0.140 0.25" joint_rpy="0 0 0"
-        parent="base_link" />
+        parent="base_link"
+        collision_xyz="-0.135 0 0.025" collision_rpy="0 0 0" collision_size="0.270 0.120 0.05"
+        mass="0.93983878"
+        ixx="0.00318358" ixy="0" ixz="0"
+        iyy="0.00133395" iyz="0.00023839" izz="0.0040904" />
     <!-- LiDAR Sensor -->
     <xacro:fixed_link
@@ -92,4 +100,8 @@
         mesh_name="${lidar_sensor}"
         joint_xyz="-0.2 0 0.05" joint_rpy="0 0 0"
-        parent="lidar_base" />
+        parent="lidar_base"
+        collision_xyz="0 0 0.0375" collision_rpy="0 0 0" collision_size="0.105 0.105 0.075"
+        mass="0.61826506"
+        ixx="0.00067265" ixy="0" ixz="0"
+        iyy="0.0006728" iyz="0" izz="0.00080351"/>
 </robot>

File: cluerosity_description/urdf/cluerosity_links.xacro (robot description, xacro)
@@ -6,9 +6,17 @@
         +==========================+
     -->
-    <xacro:macro name="fixed_link" params="name link_xyz link_rpy mesh_name joint_xyz joint_rpy parent">
+    <xacro:macro name="fixed_link" params="name link_xyz link_rpy joint_xyz joint_rpy mesh_name collision_xyz collision_rpy collision_size mass ixx ixy ixz iyy iyz izz parent">
         <link name="${name}">
             <xacro:mesh_link
                 xyz="${link_xyz}" rpy="${link_rpy}"
                 mesh_name="${mesh_name}"/>
+            <xacro:box_collision
+                xyz="${collision_xyz}" rpy="${collision_rpy}"
+                box_size="${collision_size}"/>
+            <xacro:link_inertia
+                xyz="${collision_xyz}" rpy="${collision_rpy}"
+                mass="${mass}"
+                ixx="${ixx}" ixy="${ixy}" ixz="${ixz}"
+                iyy="${iyy}" iyz="${iyz}" izz="${izz}"/>
         </link>
         <joint name="${name}_joint" type="fixed">
@@ -45,8 +53,8 @@
         <!-- Base footprint is on the ground under the robot -->
         <link name="base_footprint" />
-        <joint name="base_footprint_joint" type="fixed">
-            <origin xyz="0 0 -0.14" rpy="0 0 0" />
-            <parent link="base_link" />
-            <child link="base_footprint" />
+        <joint name="base_link_joint" type="fixed">
+            <origin xyz="0 0 0.115" rpy="0 0 0" />
+            <parent link="base_footprint" />
+            <child link="base_link" />
         </joint>
     </xacro:macro>
@@ -63,4 +71,12 @@
                 box_size="0.1 0.1 0.05"
                 material_name="dark_gray"/>
+            <xacro:box_collision
+                xyz="0 0 0.025" rpy="0 0 0"
+                box_size="0.1 0.1 0.05"/>
+            <xacro:link_inertia
+                xyz="0 0 0.025" rpy="0 0 0"
+                mass="3.4875"
+                ixx="0.004" ixy="0" ixz="0"
+                iyy="0.004" iyz="0"  izz="0.006"/>
         </link>
         <joint name="gimbal_base_joint" type="fixed">
@@ -76,4 +92,12 @@
                 xyz="0 0 0" rpy="0 0 0"
                 mesh_name="${mesh_name}"/>
+            <xacro:box_collision
+                xyz="0 0 0.12" rpy="0 0 0"
+                box_size="0.07 0.07 0.190"/>
+            <xacro:link_inertia
+                xyz="0 0 0.12" rpy="0 0 0"
+                mass="0.86030554"
+                ixx="0.00159531" ixy="0" ixz="0"
+                iyy="0.00204855" iyz="0"  izz="0.00078318"/>
         </link>
         <joint name="gimbal_axle_joint" type="continuous">
@@ -90,4 +114,12 @@
                 xyz="0 0 0.053" rpy="0 0 0"
                 mesh_name="${mesh_name}"/>
+            <xacro:box_collision
+                xyz="0 0 0.105" rpy="0 0 0"
+                box_size="0.200 0.100 0.150"/>
+            <xacro:link_inertia
+                xyz="0 0 0.105" rpy="0 0 0"
+                mass="2.14582602"
+                ixx="0.00498945" ixy="-0.00002479" ixz="0.0002252"
+                iyy="0.00883757" iyz="-0.00005538"  izz="0.00675851"/>
         </link>
         <joint name="sensor_housing_joint" type="revolute">

File: cluerosity_description/urdf/wheels.xacro (robot description, xacro)
@@ -41,4 +41,12 @@
                 radius="0.010" length="0.550"
                 material_name="white"/>
+            <xacro:cylinder_collision
+                xyz="0 0 0" rpy="${PI/2} 0 0"
+                radius="0.010" length="0.550"/>
+            <xacro:link_inertia
+                xyz="0 0 0" rpy="${PI/2} 0 0"
+                mass="0.30129837"
+                ixx="0.00759711" ixy="0" ixz="0"
+                iyy="0.00759711" iyz="0"  izz="0.00000377"/>
         </link>
         <joint name="${name}_joint" type="fixed">

Commit message: :white_check_mark: <tested ok> added the gazebo plugin to enable the drive control, camera and laser sensor work and publish the required corresponding messages

File: cluerosity_description/urdf/cluerosity.xacro (robot description, xacro)
@@ -8,4 +8,5 @@
     <xacro:include filename="$(find cluerosity_description)/urdf/wheels.xacro" />
     <xacro:include filename="$(find cluerosity_description)/urdf/cluerosity_links.xacro" />
+    <xacro:include filename="$(find cluerosity_description)/urdf/cluerosity.gazebo" />
     <!-- Properties -->
     <xacro:property name="PI" value="3.14159265359" />
@@ -78,4 +79,12 @@
         ixx="0.0000978" ixy="0" ixz="0"
         iyy="0.0000978" iyz="0" izz="0.0000491"/>
+    <!-- Camera Sensor -->
+    <xacro:sensor_link
+        name="camera_link"
+        joint_xyz="0.035 -0.05 0.125" joint_rpy="0 0 ${-PI/2}" />
+    <!-- Hokuyo Laser Scanner -->
+    <xacro:sensor_link
+        name="hokuyo_link"
+        joint_xyz="0.05 -0.05 0.035" joint_rpy="0 0 ${-PI/2}" />
     <!--
         +=======================+

File: cluerosity_description/urdf/cluerosity_links.xacro (robot description, xacro)
@@ -101,9 +101,9 @@
                 iyy="0.00204855" iyz="0"  izz="0.00078318"/>
         </link>
-        <joint name="gimbal_axle_joint" type="continuous">
+        <joint name="gimbal_axle_joint" type="fixed">  <!-- change back to "continuous" -->
             <parent link="gimbal_base" />
             <child link="gimbal_axle" />
             <origin xyz="0 0 0" rpy="0 0 0" />
-            <axis xyz="0 0 1" rpy="0 0 0" />
+            <!-- <axis xyz="0 0 1" rpy="0 0 0" /> -->
         </joint>
     </xacro:macro>
@@ -123,10 +123,32 @@
                 iyy="0.00883757" iyz="-0.00005538"  izz="0.00675851"/>
         </link>
-        <joint name="sensor_housing_joint" type="revolute">
+        <joint name="sensor_housing_joint" type="fixed"> <!-- change back to "revolute" -->
             <parent link="stepper_motor" />
             <child link="sensor_housing" />
             <origin xyz="0.122 0 0" rpy="0 0 0" />
-            <axis xyz="1 0 0" rpy="0 0 0" />
-            <limit effort="1000.0" lower="-0.35" upper="0.35" velocity="0.5" />
+            <!-- <axis xyz="1 0 0" rpy="0 0 0" />
+            <limit effort="1000.0" lower="-0.35" upper="0.35" velocity="0.5" /> -->
+        </joint>
+    </xacro:macro>
+    <!-- Sensor Link -->
+    <xacro:macro name="sensor_link" params="name joint_xyz joint_rpy">
+        <link name="${name}">
+            <xacro:box_link
+                xyz="0 0 0" rpy="0 0 0"
+                box_size="0.01 0.01 0.01"
+                material_name="dark_gray"/>
+            <xacro:box_collision
+                xyz="0 0 0" rpy="0 0 0"
+                box_size="0.01 0.01 0.01"/>
+            <xacro:link_inertia
+                xyz="0 0 0" rpy="0 0 0"
+                mass="0.1"
+                ixx="0.004" ixy="0" ixz="0"
+                iyy="0.004" iyz="0"  izz="0.006"/>
+        </link>
+        <joint name="${name}_joint" type="fixed">
+            <parent link="sensor_housing" />
+            <child link="${name}" />
+            <origin xyz="${joint_xyz}" rpy="${joint_rpy}" />
         </joint>
     </xacro:macro>

Commit message: :construction: <updated> added rgb-d camera gazebo plugin to the sensor housing

File: cluerosity_description/urdf/cluerosity.xacro (robot description, xacro)
@@ -82,9 +82,16 @@
     <xacro:sensor_link
         name="camera_link"
-        joint_xyz="0.035 -0.05 0.125" joint_rpy="0 0 ${-PI/2}" />
+        joint_xyz="0.035 -0.05 0.125" joint_rpy="0 0 ${-PI/2}"
+        parent="sensor_housing" />
+    <!-- RGB-D Camera  -->
+    <xacro:sensor_link
+        name="camera_depth_link"
+        joint_xyz="0.05 0 0" joint_rpy="${-PI/2} 0 ${-PI/2}"
+        parent="camera_link"/>
     <!-- Hokuyo Laser Scanner -->
     <xacro:sensor_link
         name="hokuyo_link"
-        joint_xyz="0.05 -0.05 0.035" joint_rpy="0 0 ${-PI/2}" />
+        joint_xyz="0.05 -0.05 0.035" joint_rpy="0 0 ${-PI/2}"
+        parent="sensor_housing" />
     <!--
         +=======================+

File: cluerosity_description/urdf/cluerosity_links.xacro (robot description, xacro)
@@ -132,5 +132,5 @@
     </xacro:macro>
     <!-- Sensor Link -->
-    <xacro:macro name="sensor_link" params="name joint_xyz joint_rpy">
+    <xacro:macro name="sensor_link" params="name joint_xyz joint_rpy parent">
         <link name="${name}">
             <xacro:box_link
@@ -148,5 +148,5 @@
         </link>
         <joint name="${name}_joint" type="fixed">
-            <parent link="sensor_housing" />
+            <parent link="${parent}" />
             <child link="${name}" />
             <origin xyz="${joint_xyz}" rpy="${joint_rpy}" />
