Commit message: :white_check_mark: <added> robot description of the cluerosity manipulator

File: cluerosity_description/urdf/cluerosity.xacro (robot description, xacro)
@@ -121,3 +121,108 @@
         ixx="0.00067265" ixy="0" ixz="0"
         iyy="0.0006728" iyz="0" izz="0.00080351"/>
+    <!--
+        +=======================+
+        |       Manipulator      |
+        +=======================+
+    -->
+    <xacro:fixed_link
+    name="motor_01"
+    link_xyz="0 0 0" link_rpy="0 0 0"
+    mesh_name="${motor}"
+    joint_xyz="0.498 0.15 0.09" joint_rpy="${PI} 0 0"
+    parent="base_link"
+    collision_xyz="0 0 0" collision_rpy="0 0 0" collision_size="0.105 0.105 0.075"
+    mass="0.61826506"
+    ixx="0.00067265" ixy="0" ixz="0"
+    iyy="0.0006728" iyz="0" izz="0.00080351"/>
+    <xacro:fixed_link
+    name="motor_connector_01"
+    link_xyz="0 0 0" link_rpy="0 0 0"
+    mesh_name="${motor_connector_01}"
+    joint_xyz="0.046 0 0.0395" joint_rpy="${PI/2} ${PI/2} 0"
+    parent="motor_01"
+    collision_xyz="0 0 0" collision_rpy="0 0 0" collision_size="0.105 0.105 0.075"
+    mass="0.61826506"
+    ixx="0.00067265" ixy="0" ixz="0"
+    iyy="0.0006728" iyz="0" izz="0.00080351"/>
+    <xacro:fixed_link
+    name="motor_02"
+    link_xyz="0 0 0" link_rpy="0 0 0"
+    mesh_name="${motor}"
+    joint_xyz="0 0.036 -0.0395" joint_rpy="0 0 0"
+    parent="motor_connector_01"
+    collision_xyz="0 0 0" collision_rpy="0 0 0" collision_size="0.105 0.105 0.075"
+    mass="0.61826506"
+    ixx="0.00067265" ixy="0" ixz="0"
+    iyy="0.0006728" iyz="0" izz="0.00080351"/>
+    <xacro:fixed_link
+    name="link_01"
+    link_xyz="0 0 0" link_rpy="0 0 0"
+    mesh_name="${link_01}"
+    joint_xyz="0 0 0" joint_rpy="0 0 ${PI}"
+    parent="motor_02"
+    collision_xyz="0 0 0" collision_rpy="0 0 0" collision_size="0.105 0.105 0.075"
+    mass="0.61826506"
+    ixx="0.00067265" ixy="0" ixz="0"
+    iyy="0.0006728" iyz="0" izz="0.00080351"/>
+    <xacro:fixed_link
+    name="motor_03"
+    link_xyz="0 0 0" link_rpy="0 0 0"
+    mesh_name="${motor}"
+    joint_xyz="0 -0.35 0" joint_rpy="0 0 0"
+    parent="link_01"
+    collision_xyz="0 0 0" collision_rpy="0 0 0" collision_size="0.105 0.105 0.075"
+    mass="0.61826506"
+    ixx="0.00067265" ixy="0" ixz="0"
+    iyy="0.0006728" iyz="0" izz="0.00080351"/>
+    <xacro:fixed_link
+    name="link_02"
+    link_xyz="0 0 0" link_rpy="0 0 0"
+    mesh_name="${link_02}"
+    joint_xyz="0 0 0.0395" joint_rpy="0 0 ${PI}"
+    parent="motor_03"
+    collision_xyz="0 0 0" collision_rpy="0 0 0" collision_size="0.105 0.105 0.075"
+    mass="0.61826506"
+    ixx="0.00067265" ixy="0" ixz="0"
+    iyy="0.0006728" iyz="0" izz="0.00080351"/>
+    <xacro:fixed_link
+    name="motor_04"
+    link_xyz="0 0 0" link_rpy="0 0 0"
+    mesh_name="${motor}"
+    joint_xyz="0.370 0 -0.0395" joint_rpy="0 0 0"
+    parent="link_02"
+    collision_xyz="0 0 0" collision_rpy="0 0 0" collision_size="0.105 0.105 0.075"
+    mass="0.61826506"
+    ixx="0.00067265" ixy="0" ixz="0"
+    iyy="0.0006728" iyz="0" izz="0.00080351"/>
+    <xacro:fixed_link
+    name="motor_connector_02"
+    link_xyz="0 0 0" link_rpy="0 0 0"
+    mesh_name="${motor_connector_02}"
+    joint_xyz="0 0 0" joint_rpy="0 0 0"
+    parent="motor_04"
+    collision_xyz="0 0 0" collision_rpy="0 0 0" collision_size="0.105 0.105 0.075"
+    mass="0.61826506"
+    ixx="0.00067265" ixy="0" ixz="0"
+    iyy="0.0006728" iyz="0" izz="0.00080351"/>
+    <xacro:fixed_link
+    name="motor_05"
+    link_xyz="0 0 0" link_rpy="0 0 0"
+    mesh_name="${motor}"
+    joint_xyz="0.1395 0 0.1" joint_rpy="0 ${-PI/2} 0"
+    parent="motor_connector_02"
+    collision_xyz="0 0 0" collision_rpy="0 0 0" collision_size="0.105 0.105 0.075"
+    mass="0.61826506"
+    ixx="0.00067265" ixy="0" ixz="0"
+    iyy="0.0006728" iyz="0" izz="0.00080351"/>
+    <xacro:fixed_link
+    name="end_effector_connector"
+    link_xyz="0 0 0" link_rpy="0 0 0"
+    mesh_name="${end_effector_connector}"
+    joint_xyz="0 0 0" joint_rpy="0 0 ${-PI/2}"
+    parent="motor_05"
+    collision_xyz="0 0 0" collision_rpy="0 0 0" collision_size="0.105 0.105 0.075"
+    mass="0.61826506"
+    ixx="0.00067265" ixy="0" ixz="0"
+    iyy="0.0006728" iyz="0" izz="0.00080351"/>
 </robot>

File: cluerosity_description/urdf/cluerosity_links.xacro (robot description, xacro)
@@ -134,5 +134,5 @@
     <xacro:macro name="sensor_link" params="name joint_xyz joint_rpy parent">
         <link name="${name}">
-            <xacro:box_link
+            <!-- <xacro:box_link
                 xyz="0 0 0" rpy="0 0 0"
                 box_size="0.01 0.01 0.01"
@@ -145,5 +145,5 @@
                 mass="0.1"
                 ixx="0.004" ixy="0" ixz="0"
-                iyy="0.004" iyz="0"  izz="0.006"/>
+                iyy="0.004" iyz="0"  izz="0.006"/> -->
         </link>
         <joint name="${name}_joint" type="fixed">

File: cluerosity_description/urdf/meshes.xacro (robot description, xacro)
@@ -9,3 +9,9 @@
     <xacro:property name="lidar_base" value="package://cluerosity_description/meshes/lidar_base.dae" />
     <xacro:property name="lidar_sensor" value="package://cluerosity_description/meshes/velodyne_lidar.dae" />
+    <xacro:property name="motor" value="package://cluerosity_description/meshes/motor.dae" />
+    <xacro:property name="motor_connector_01" value="package://cluerosity_description/meshes/motor_connector_01.dae" />
+    <xacro:property name="motor_connector_02" value="package://cluerosity_description/meshes/motor_connector_02.dae" />
+    <xacro:property name="link_01" value="package://cluerosity_description/meshes/link_01.dae" />
+    <xacro:property name="link_02" value="package://cluerosity_description/meshes/link_02.dae" />
+    <xacro:property name="end_effector_connector" value="package://cluerosity_description/meshes/end_effector_connector.dae" />
 </robot>

Commit message: :construction: <updated> added mobility to the robot manipulator

File: cluerosity_description/urdf/cluerosity.xacro (robot description, xacro)
@@ -121,108 +121,3 @@
         ixx="0.00067265" ixy="0" ixz="0"
         iyy="0.0006728" iyz="0" izz="0.00080351"/>
-    <!--
-        +=======================+
-        |       Manipulator      |
-        +=======================+
-    -->
-    <xacro:fixed_link
-    name="motor_01"
-    link_xyz="0 0 0" link_rpy="0 0 0"
-    mesh_name="${motor}"
-    joint_xyz="0.498 0.15 0.09" joint_rpy="${PI} 0 0"
-    parent="base_link"
-    collision_xyz="0 0 0" collision_rpy="0 0 0" collision_size="0.105 0.105 0.075"
-    mass="0.61826506"
-    ixx="0.00067265" ixy="0" ixz="0"
-    iyy="0.0006728" iyz="0" izz="0.00080351"/>
-    <xacro:fixed_link
-    name="motor_connector_01"
-    link_xyz="0 0 0" link_rpy="0 0 0"
-    mesh_name="${motor_connector_01}"
-    joint_xyz="0.046 0 0.0395" joint_rpy="${PI/2} ${PI/2} 0"
-    parent="motor_01"
-    collision_xyz="0 0 0" collision_rpy="0 0 0" collision_size="0.105 0.105 0.075"
-    mass="0.61826506"
-    ixx="0.00067265" ixy="0" ixz="0"
-    iyy="0.0006728" iyz="0" izz="0.00080351"/>
-    <xacro:fixed_link
-    name="motor_02"
-    link_xyz="0 0 0" link_rpy="0 0 0"
-    mesh_name="${motor}"
-    joint_xyz="0 0.036 -0.0395" joint_rpy="0 0 0"
-    parent="motor_connector_01"
-    collision_xyz="0 0 0" collision_rpy="0 0 0" collision_size="0.105 0.105 0.075"
-    mass="0.61826506"
-    ixx="0.00067265" ixy="0" ixz="0"
-    iyy="0.0006728" iyz="0" izz="0.00080351"/>
-    <xacro:fixed_link
-    name="link_01"
-    link_xyz="0 0 0" link_rpy="0 0 0"
-    mesh_name="${link_01}"
-    joint_xyz="0 0 0" joint_rpy="0 0 ${PI}"
-    parent="motor_02"
-    collision_xyz="0 0 0" collision_rpy="0 0 0" collision_size="0.105 0.105 0.075"
-    mass="0.61826506"
-    ixx="0.00067265" ixy="0" ixz="0"
-    iyy="0.0006728" iyz="0" izz="0.00080351"/>
-    <xacro:fixed_link
-    name="motor_03"
-    link_xyz="0 0 0" link_rpy="0 0 0"
-    mesh_name="${motor}"
-    joint_xyz="0 -0.35 0" joint_rpy="0 0 0"
-    parent="link_01"
-    collision_xyz="0 0 0" collision_rpy="0 0 0" collision_size="0.105 0.105 0.075"
-    mass="0.61826506"
-    ixx="0.00067265" ixy="0" ixz="0"
-    iyy="0.0006728" iyz="0" izz="0.00080351"/>
-    <xacro:fixed_link
-    name="link_02"
-    link_xyz="0 0 0" link_rpy="0 0 0"
-    mesh_name="${link_02}"
-    joint_xyz="0 0 0.0395" joint_rpy="0 0 ${PI}"
-    parent="motor_03"
-    collision_xyz="0 0 0" collision_rpy="0 0 0" collision_size="0.105 0.105 0.075"
-    mass="0.61826506"
-    ixx="0.00067265" ixy="0" ixz="0"
-    iyy="0.0006728" iyz="0" izz="0.00080351"/>
-    <xacro:fixed_link
-    name="motor_04"
-    link_xyz="0 0 0" link_rpy="0 0 0"
-    mesh_name="${motor}"
-    joint_xyz="0.370 0 -0.0395" joint_rpy="0 0 0"
-    parent="link_02"
-    collision_xyz="0 0 0" collision_rpy="0 0 0" collision_size="0.105 0.105 0.075"
-    mass="0.61826506"
-    ixx="0.00067265" ixy="0" ixz="0"
-    iyy="0.0006728" iyz="0" izz="0.00080351"/>
-    <xacro:fixed_link
-    name="motor_connector_02"
-    link_xyz="0 0 0" link_rpy="0 0 0"
-    mesh_name="${motor_connector_02}"
-    joint_xyz="0 0 0" joint_rpy="0 0 0"
-    parent="motor_04"
-    collision_xyz="0 0 0" collision_rpy="0 0 0" collision_size="0.105 0.105 0.075"
-    mass="0.61826506"
-    ixx="0.00067265" ixy="0" ixz="0"
-    iyy="0.0006728" iyz="0" izz="0.00080351"/>
-    <xacro:fixed_link
-    name="motor_05"
-    link_xyz="0 0 0" link_rpy="0 0 0"
-    mesh_name="${motor}"
-    joint_xyz="0.1395 0 0.1" joint_rpy="0 ${-PI/2} 0"
-    parent="motor_connector_02"
-    collision_xyz="0 0 0" collision_rpy="0 0 0" collision_size="0.105 0.105 0.075"
-    mass="0.61826506"
-    ixx="0.00067265" ixy="0" ixz="0"
-    iyy="0.0006728" iyz="0" izz="0.00080351"/>
-    <xacro:fixed_link
-    name="end_effector_connector"
-    link_xyz="0 0 0" link_rpy="0 0 0"
-    mesh_name="${end_effector_connector}"
-    joint_xyz="0 0 0" joint_rpy="0 0 ${-PI/2}"
-    parent="motor_05"
-    collision_xyz="0 0 0" collision_rpy="0 0 0" collision_size="0.105 0.105 0.075"
-    mass="0.61826506"
-    ixx="0.00067265" ixy="0" ixz="0"
-    iyy="0.0006728" iyz="0" izz="0.00080351"/>
 </robot>

File: cluerosity_description/urdf/cluerosity_links.xacro (robot description, xacro)
@@ -24,4 +24,57 @@
             <child link="${name}" />
             <origin xyz="${joint_xyz}" rpy="${joint_rpy}" />
+        </joint>
+    </xacro:macro>
+    <!--
+        +===========================+
+        |   Continuous Link Macro    |
+        +==========================+
+    -->
+    <xacro:macro name="continuous_link" params="name link_xyz link_rpy joint_xyz joint_rpy mesh_name collision_xyz collision_rpy collision_size mass ixx ixy ixz iyy iyz izz parent axis_xyz axis_rpy">
+        <link name="${name}">
+            <xacro:mesh_link
+                xyz="${link_xyz}" rpy="${link_rpy}"
+                mesh_name="${mesh_name}"/>
+            <xacro:box_collision
+                xyz="${collision_xyz}" rpy="${collision_rpy}"
+                box_size="${collision_size}"/>
+            <xacro:link_inertia
+                xyz="${collision_xyz}" rpy="${collision_rpy}"
+                mass="${mass}"
+                ixx="${ixx}" ixy="${ixy}" ixz="${ixz}"
+                iyy="${iyy}" iyz="${iyz}" izz="${izz}"/>
+        </link>
+        <joint name="${name}_joint" type="continuous">
+            <parent link="${parent}" />
+            <child link="${name}" />
+            <origin xyz="${joint_xyz}" rpy="${joint_rpy}" />
+            <axis xyz="${axis_xyz}" rpy="${axis_rpy}" />
+        </joint>
+    </xacro:macro>
+    <!--
+        +===========================+
+        |  Revolute Link Macro    |
+        +==========================+
+    -->
+    <xacro:macro name="revolute_link" params="name link_xyz link_rpy joint_xyz joint_rpy mesh_name collision_xyz collision_rpy collision_size mass ixx ixy ixz iyy iyz izz parent axis_xyz axis_rpy lower upper">
+        <link name="${name}">
+            <xacro:mesh_link
+                xyz="${link_xyz}" rpy="${link_rpy}"
+                mesh_name="${mesh_name}"/>
+            <xacro:box_collision
+                xyz="${collision_xyz}" rpy="${collision_rpy}"
+                box_size="${collision_size}"/>
+            <xacro:link_inertia
+                xyz="${collision_xyz}" rpy="${collision_rpy}"
+                mass="${mass}"
+                ixx="${ixx}" ixy="${ixy}" ixz="${ixz}"
+                iyy="${iyy}" iyz="${iyz}" izz="${izz}"/>
+        </link>
+        <joint name="${name}_joint" type="revolute">
+            <parent link="${parent}" />
+            <child link="${name}" />
+            <origin xyz="${joint_xyz}" rpy="${joint_rpy}" />
+            <axis xyz="${axis_xyz}" rpy="${axis_rpy}" />
+            <limit effort="1000.0" lower="${lower}" upper="${upper}" velocity="0.5" /> -->
         </joint>
     </xacro:macro>

Commit message: :construction: <working ok> added controller to the sensor housing and tuned it...

File: cluerosity_description/urdf/cluerosity.xacro (robot description, xacro)
@@ -121,3 +121,23 @@
         ixx="0.00067265" ixy="0" ixz="0"
         iyy="0.0006728" iyz="0" izz="0.00080351"/>
+        <transmission name="sensor_housing_trans">
+            <type>transmission_interface/SimpleTransmission</type>
+            <joint name="sensor_housing_joint">
+                <hardwareInterface>hardware_interface/EffortJointInterface</hardwareInterface>
+            </joint>
+            <actuator name="motor7">
+                <hardwareInterface>hardware_interface/EffortJointInterface</hardwareInterface>
+                <mechanicalInterface>1</mechanicalInterface>
+            </actuator>
+        </transmission>
+        <transmission name="gimbal_axle_trans">
+            <type>transmission_interface/SimpleTransmission</type>
+            <joint name="gimbal_axle_joint">
+                <hardwareInterface>hardware_interface/EffortJointInterface</hardwareInterface>
+            </joint>
+            <actuator name="motor6">
+                <hardwareInterface>hardware_interface/EffortJointInterface</hardwareInterface>
+                <mechanicalInterface>1</mechanicalInterface>
+            </actuator>
+        </transmission>
 </robot>

File: cluerosity_description/urdf/cluerosity_links.xacro (robot description, xacro)
@@ -154,9 +154,9 @@
                 iyy="0.00204855" iyz="0"  izz="0.00078318"/>
         </link>
-        <joint name="gimbal_axle_joint" type="fixed">  <!-- change back to "continuous" -->
+        <joint name="gimbal_axle_joint" type="continuous">  <!-- change back to "continuous" -->
             <parent link="gimbal_base" />
             <child link="gimbal_axle" />
             <origin xyz="0 0 0" rpy="0 0 0" />
-            <!-- <axis xyz="0 0 1" rpy="0 0 0" /> -->
+            <axis xyz="0 0 1" rpy="0 0 0" />
         </joint>
     </xacro:macro>
@@ -176,10 +176,10 @@
                 iyy="0.00883757" iyz="-0.00005538"  izz="0.00675851"/>
         </link>
-        <joint name="sensor_housing_joint" type="fixed"> <!-- change back to "revolute" -->
+        <joint name="sensor_housing_joint" type="revolute"> <!-- change back to "revolute" -->
             <parent link="stepper_motor" />
             <child link="sensor_housing" />
             <origin xyz="0.122 0 0" rpy="0 0 0" />
-            <!-- <axis xyz="1 0 0" rpy="0 0 0" />
-            <limit effort="1000.0" lower="-0.35" upper="0.35" velocity="0.5" /> -->
+            <axis xyz="1 0 0" rpy="0 0 0" />
+            <limit effort="1000.0" lower="-0.35" upper="0.35" velocity="0.5" />
         </joint>
     </xacro:macro>

Commit message: :white_check_mark: :bug: <fixed bug> in moveit gazebo launch files and controller config

File: cluerosity_description/urdf/cluerosity.xacro (robot description, xacro)
@@ -9,4 +9,5 @@
     <xacro:include filename="$(find cluerosity_description)/urdf/cluerosity_links.xacro" />
     <xacro:include filename="$(find cluerosity_description)/urdf/cluerosity.gazebo" />
+    <xacro:include filename="$(find cluerosity_description)/urdf/gimbal_transmission.xacro" />
     <!-- Properties -->
     <xacro:property name="PI" value="3.14159265359" />
@@ -121,23 +122,3 @@
         ixx="0.00067265" ixy="0" ixz="0"
         iyy="0.0006728" iyz="0" izz="0.00080351"/>
-        <transmission name="sensor_housing_trans">
-            <type>transmission_interface/SimpleTransmission</type>
-            <joint name="sensor_housing_joint">
-                <hardwareInterface>hardware_interface/EffortJointInterface</hardwareInterface>
-            </joint>
-            <actuator name="motor7">
-                <hardwareInterface>hardware_interface/EffortJointInterface</hardwareInterface>
-                <mechanicalInterface>1</mechanicalInterface>
-            </actuator>
-        </transmission>
-        <transmission name="gimbal_axle_trans">
-            <type>transmission_interface/SimpleTransmission</type>
-            <joint name="gimbal_axle_joint">
-                <hardwareInterface>hardware_interface/EffortJointInterface</hardwareInterface>
-            </joint>
-            <actuator name="motor6">
-                <hardwareInterface>hardware_interface/EffortJointInterface</hardwareInterface>
-                <mechanicalInterface>1</mechanicalInterface>
-            </actuator>
-        </transmission>
 </robot>

File: cluerosity_description/urdf/cluerosity_manipulator.xacro (robot description, xacro)
@@ -2,6 +2,125 @@
 <robot name="cluerosity_manipulator" xmlns:xacro="http://www.ros.org/wiki/xacro">
     <!-- Includes -->
-    <xacro:include filename="$(find cluerosity_description)/urdf/cluerosity.xacro" />
-    <xacro:include filename="$(find cluerosity_description)/urdf/transmission.xacro" />
+    <xacro:include filename="$(find cluerosity_description)/urdf/meshes.xacro" />
+    <xacro:include filename="$(find cluerosity_description)/urdf/materials.xacro" />
+    <xacro:include filename="$(find cluerosity_description)/urdf/visual.xacro" />
+    <xacro:include filename="$(find cluerosity_description)/urdf/physics.xacro" />
+    <xacro:include filename="$(find cluerosity_description)/urdf/wheels.xacro" />
+    <xacro:include filename="$(find cluerosity_description)/urdf/cluerosity_links.xacro" />
+    <xacro:include filename="$(find cluerosity_description)/urdf/cluerosity.gazebo" />
+    <xacro:include filename="$(find cluerosity_description)/urdf/manipulator_transmission.xacro" />
+    <xacro:include filename="$(find cluerosity_description)/urdf/gimbal_transmission.xacro" />
+    <!-- Properties -->
+    <xacro:property name="PI" value="3.14159265359" />
+    <!--
+        +=====================+
+        |      Base Link      |
+        +=====================+
+    -->
+    <xacro:base_link mesh_name="${robot_base}"/>
+    <!--
+        +=====================+
+        |     Wheel Shaft     |
+        +=====================+
+    -->
+    <xacro:cluerosity_shaft
+        name="front_shaft"
+        joint_xyz="0.350 0 0.05" />
+    <xacro:cluerosity_shaft
+        name="rear_shaft"
+        joint_xyz="-0.20 0 0.05" />
+    <!--
+        +=====================+
+        |   Wheel definition  |
+        +=====================+
+    -->
+    <!-- Right Front Wheel -->
+    <xacro:cluerosity_wheel
+        name="right_front_wheel"
+        tyre_xyz="-0.14686986 0 0" tyre_rpy="${PI/2} 0 ${-PI/2}"
+        rim_xyz="0 0 0" rim_rpy="0 0 0"
+        joint_xyz="0.35 -0.30 0.05" joint_rpy="0 0 0" />
+    <!-- Right Rear Wheel -->
+    <xacro:cluerosity_wheel
+        name="right_rear_wheel"
+        tyre_xyz="-0.14686986 0 0" tyre_rpy="${PI/2} 0 ${-PI/2}"
+        rim_xyz="0 0 0" rim_rpy="0 0 0"
+        joint_xyz="-0.20 -0.30 0.05" joint_rpy="0 0 0" />
+    <!-- Left Front Wheel -->
+    <xacro:cluerosity_wheel
+        name="left_front_wheel"
+        tyre_xyz="-0.14686986 0 0" tyre_rpy="${PI/2} 0 ${-PI/2}"
+        rim_xyz="0 0 0" rim_rpy="0 0 ${PI}"
+        joint_xyz="0.35 0.30 0.05" joint_rpy="0 0 0" />
+    <!-- Left Rear Wheel -->
+    <xacro:cluerosity_wheel
+        name="left_rear_wheel"
+        tyre_xyz="-0.14686986 0 0" tyre_rpy="${PI/2} 0 ${-PI/2}"
+        rim_xyz="0 0 0" rim_rpy="0 0 ${PI}"
+        joint_xyz="-0.20 0.30 0.05" joint_rpy="0 0 0" />
+    <!--
+        +=====================+
+        |   Sensor Gimbal     |
+        +=====================+
+    -->
+    <!-- Gimbal Base  -->
+    <xacro:gimbal_base />
+    <!-- Gimbal Axle  -->
+    <xacro:gimbal_axle mesh_name="${gimbal_axle}"/>
+    <!-- Gimbal Sensor Housing  -->
+    <xacro:sensor_housing mesh_name="${sensor_housing}" />
+    <!-- Stepper Motor -->
+    <xacro:fixed_link
+        name="stepper_motor"
+        link_xyz="0 0 0" link_rpy="0 ${PI/2} 0"
+        mesh_name="${stepper_motor}"
+        joint_xyz="-0.10 0 0.19" joint_rpy="0 0 0"
+        parent="gimbal_axle"
+        collision_xyz="0.0325 0 0" collision_rpy="0 ${PI/2} 0" collision_size="0.05 0.05 0.080"
+        mass="0.20879833"
+        ixx="0.0000978" ixy="0" ixz="0"
+        iyy="0.0000978" iyz="0" izz="0.0000491"/>
+    <!-- Camera Sensor -->
+    <xacro:sensor_link
+        name="camera_link"
+        joint_xyz="0.035 -0.05 0.125" joint_rpy="0 0 ${-PI/2}"
+        parent="sensor_housing" />
+    <!-- RGB-D Camera  -->
+    <xacro:sensor_link
+        name="camera_depth_link"
+        joint_xyz="0.05 0 0" joint_rpy="${-PI/2} 0 ${-PI/2}"
+        parent="camera_link"/>
+    <!-- Hokuyo Laser Scanner -->
+    <xacro:sensor_link
+        name="hokuyo_link"
+        joint_xyz="0.05 -0.05 0.035" joint_rpy="0 0 ${-PI/2}"
+        parent="sensor_housing" />
+    <!--
+        +=======================+
+        | Velodyne LiDAR Sensor |
+        +=======================+
+    -->
+    <!-- LiDAR Base -->
+    <xacro:fixed_link
+        name="lidar_base"
+        link_xyz="-0.075 0 0.05" link_rpy="0 ${PI} ${PI/2}"
+        mesh_name="${lidar_base}"
+        joint_xyz="-0.325 0.140 0.25" joint_rpy="0 0 0"
+        parent="base_link"
+        collision_xyz="-0.135 0 0.025" collision_rpy="0 0 0" collision_size="0.270 0.120 0.05"
+        mass="0.93983878"
+        ixx="0.00318358" ixy="0" ixz="0"
+        iyy="0.00133395" iyz="0.00023839" izz="0.0040904" />
+    <!-- LiDAR Sensor -->
+    <xacro:fixed_link
+        name="lidar_sensor"
+        link_xyz="0 0 0" link_rpy="0 0 0"
+        mesh_name="${lidar_sensor}"
+        joint_xyz="-0.2 0 0.05" joint_rpy="0 0 0"
+        parent="lidar_base"
+        collision_xyz="0 0 0.0375" collision_rpy="0 0 0" collision_size="0.105 0.105 0.075"
+        mass="0.61826506"
+        ixx="0.00067265" ixy="0" ixz="0"
+        iyy="0.0006728" iyz="0" izz="0.00080351"/>
     <!--
         +=======================+
